File: etched-disco-board-pcb/disco-board-pcb.kicad_pcb (KiCad board)
At the start: 2 copper layers, 57.2 x 82.6 mm, 15 parts, among them J1 Conn_02x32_Odd_Even, J2 Conn_02x32_Odd_Even, U2 MMA8452Q

Commit message: Correcting error in PCB where NRST was connected to GND on etched-disco-board-pcb
Connections:
- J2 pad 12: GND -> unconnected-(J2-Pad12)
- J2 pad 30: GND -> unconnected-(J2-Pad30)
Changed lines of the file:
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@@
   (net 128 "unconnected-(U2-Pad15)")
   (net 129 "unconnected-(U2-Pad16)")
+  (net 130 "unconnected-(J2-Pad12)")
+  (net 131 "unconnected-(J2-Pad30)")
   (footprint "local:LPS28DFWTR" (layer "B.Cu")
     (at 39.38 87.537726 90)
@@
       (net 2 "GND") (pinfunction "Pin_11") (pintype "passive"))
     (pad "12" thru_hole oval locked (at -2.54 -12.7 180) (size 1.7 1.7) (drill 0.5) (layers *.Cu *.Mask)
-      (net 2 "GND") (pinfunction "Pin_12") (pintype "passive"))
+      (net 130 "unconnected-(J2-Pad12)") (pinfunction "Pin_12") (pintype "passive"))
     (pad "13" thru_hole oval locked (at 0 -15.24 180) (size 1.7 1.7) (drill 1) (layers *.Cu *.Mask)
       (net 80 "unconnected-(J2-Pad13)") (pinfunction "Pin_13") (pintype "passive"))
@@
       (net 2 "GND") (pinfunction "Pin_29") (pintype "passive"))
     (pad "30" thru_hole oval locked (at -2.54 -35.56 180) (size 1.7 1.7) (drill 0.5) (layers *.Cu *.Mask)
-      (net 2 "GND") (pinfunction "Pin_30") (pintype "passive"))
+      (net 131 "unconnected-(J2-Pad30)") (pinfunction "Pin_30") (pintype "passive"))
     (pad "31" thru_hole oval locked (at 0 -38.1 180) (size 1.7 1.7) (drill 1) (layers *.Cu *.Mask)
       (net 94 "unconnected-(J2-Pad31)") (pinfunction "Pin_31") (pintype "passive"))
